Commit message: wip-moveit_bridge

File: bartending_robot_description/urdf/bartending_robot_arm.urdf (robot description, URDF)
Before this commit: robot bartending_robot_arm, 6 links, 5 joints
Links:
- added link base_platform, mass 5; collision box size=0.2 0.12 0.015; visual box size=0.2 0.12 0.015
- added link gripper_link, mass 0.15; collision box size=0.05 0.11 0.1; visual box size=0.05 0.11 0.1
- link base_link: mass 3 -> 1; geometry collision box size=0.06 0.04 0.043; visual box size=0.06 0.04 0.043
- link end_effector_link: geometry collision box size=0.03 0.05 0.068; visual box size=0.03 0.05 0.068
- link lower_link: geometry collision box size=0.03 0.05 0.068; visual box size=0.03 0.05 0.068
- link upper_link: geometry collision box size=0.03 0.05 0.068; visual box size=0.03 0.05 0.068
Joints:
- added joint base_mount: type fixed, parent base_platform, child base_link, origin xyz=0.043 0 0.029
- added joint gripper_z_rot: type revolute, parent tooltip_mount, child gripper_link, origin xyz=-0.015 0 0, axis 0 0 1, limit lower=-1.734 upper=1.616 effort=0 velocity=1.0
- joint base_y_rot: limit lower=-1.311 upper=0.964 effort=0 velocity=1.0 -> lower=-1.007 upper=1.447 effort=0 velocity=1.0; origin xyz=-0.0075 0 0.025 -> xyz=-0.0075 0 0.0125
- joint base_z_rot: limit lower=-1.953 upper=1.319 effort=0 velocity=1.0 -> lower=-1.62089 upper=1.6005 effort=0 velocity=1.0; origin xyz=0 0 0.025 -> xyz=-0.011 0 0.034
- joint elbow_y_rot: limit lower=-1.734 upper=1.616 effort=0 velocity=1.0 -> lower=-1.687 upper=1.6619 effort=0 velocity=1.0; origin xyz=0 0 0.115 -> xyz=0 0 0.068
- joint gripper_mount: origin xyz=-0.012 0 0.076 -> xyz=-0.012 0 0.0825
- joint wrist_y_rot: limit lower=-2.054 upper=1.781 effort=0 velocity=1.0 -> lower=-1.713 upper=1.6413 effort=0 velocity=1.0; origin xyz=0 0 0.094 -> xyz=0 0 0.068

Commit message: saved work - can plan motion now, but with some calibrations yet to do

File: bartending_robot_description/urdf/bartending_robot_arm.urdf (robot description, URDF)
Before this commit: robot bartending_robot_arm, 8 links, 7 joints
Links:
- link base_platform: mass 5 -> None
Joints:
- joint gripper_z_rot: limit lower=-1.734 upper=1.616 effort=0 velocity=1.0 -> lower=-3.14 upper=3.14 effort=0 velocity=1.0

Commit message: added approximate ik capability. TODO: write my own ik solver

File: bartending_robot_description/urdf/bartending_robot_arm.urdf (robot description, URDF)
Before this commit: robot bartending_robot_arm, 8 links, 7 joints
Links:
- link base_link: mass 1 -> None
- link base_link_offset: mass 0.1 -> None
- link end_effector_link: mass 0.15 -> None
- link gripper_link: mass 0.15 -> None
- link lower_link: mass 0.15 -> None
- link tooltip_mount: mass 0.15 -> None
- link upper_link: mass 0.15 -> None

Commit message: saved work - moveit motion planner

File: bartending_robot_description/urdf/bartending_robot_arm.urdf (robot description, URDF)
Before this commit: robot bartending_robot_arm, 8 links, 7 joints
Joints:
- joint base_y_rot: limit lower=-1.007 upper=1.447 effort=0 velocity=1.0 -> lower=-1.007 upper=1.447 effort=0 velocity=0.2
- joint base_z_rot: limit lower=-1.62089 upper=1.6005 effort=0 velocity=1.0 -> lower=-3.14 upper=3.14 effort=0 velocity=0.2
- joint elbow_y_rot: limit lower=-1.687 upper=1.6619 effort=0 velocity=1.0 -> lower=-1.687 upper=1.6619 effort=0 velocity=0.2
- joint gripper_z_rot: limit lower=-3.14 upper=3.14 effort=0 velocity=1.0 -> lower=-3.14 upper=3.14 effort=0 velocity=0.2
- joint wrist_y_rot: limit lower=-1.713 upper=1.6413 effort=0 velocity=1.0 -> lower=-1.713 upper=1.6413 effort=0 velocity=0.2

Commit message: updated parameters and offsets

File: bartending_robot_description/urdf/bartending_robot_arm.urdf (robot description, URDF)
Before this commit: robot bartending_robot_arm, 8 links, 7 joints
Links:
- link gripper_link: geometry collision box size=0.05 0.11 0.1; visual box size=0.03 0.1 0.105

Commit message: saved work - pouring of alcohol and mixer works, but requires some tuning

File: bartending_robot_description/urdf/bartending_robot_arm.urdf (robot description, URDF)
Before this commit: robot bartending_robot_arm, 8 links, 7 joints
Links:
- added link gripper_motor; collision box size=0.001 0.001 0.001; visual box size=0.001 0.001 0.001
Joints:
- added joint gripper_actuator: type fixed, parent gripper_link, child gripper_motor, origin xyz=0.0 0 0

Commit message: changed config for robot arm

File: bartending_robot_description/urdf/bartending_robot_arm.urdf (robot description, URDF)
Before this commit: robot bartending_robot_arm, 9 links, 8 joints
Links:
- link gripper_link: geometry collision box size=0.03 0.1 0.105; visual box size=0.03 0.1 0.105

Commit message: edited urdf + some minor refactor

File: bartending_robot_description/urdf/bartending_robot_arm.urdf (robot description, URDF)
Before this commit: robot bartending_robot_arm, 9 links, 8 joints
Links:
- link end_effector_link: geometry collision box size=0.03 0.05 0.005; visual box size=0.03 0.05 0.005
- link tooltip_mount: geometry collision box size=0.078 0.05 0.038; visual box size=0.078 0.05 0.038
Joints:
- joint base_y_rot: limit lower=-1.007 upper=1.447 effort=0 velocity=0.2 -> lower=-1.825 upper=1.447 effort=100 velocity=1.1624
- joint base_z_rot: limit lower=-3.14 upper=3.14 effort=0 velocity=0.2 -> lower=-3.14 upper=3.14 effort=100 velocity=1.7436
- joint elbow_y_rot: limit lower=-1.687 upper=1.6619 effort=0 velocity=0.2 -> lower=-1.687 upper=1.6619 effort=100 velocity=1.1624
- joint gripper_z_rot: limit lower=-3.14 upper=3.14 effort=0 velocity=0.2 -> lower=-3.14 upper=3.14 effort=100 velocity=1.7436
- joint wrist_y_rot: limit lower=-1.713 upper=1.6413 effort=0 velocity=0.2 -> lower=-1.713 upper=1.6413 effort=100 velocity=1.7436
